File: 4mb mapper nms8280.kicad_pcb (KiCad board)
At the start: 2 copper layers, 102.2 x 68.2 mm, 28 parts, among them IC147 74LS157, IC147B1 74LS157, IC149 74LS670, IC149B1 74LS670, J1 Conn_01x10_Pin

Commit message: Update 4MB mapper PCB
Parts:
- renumbered C131B2 to C131C1
Routing:
- net GND: track 50.2 -> 51.6 mm, vias 27 -> 26
- net Net-(IC131B1-3O): track 56.2 -> 55.1 mm

Commit message: Update 4MB mapper design outputs
Parts:
- IC131, IC131B1, IC131C1: value ~ -> 74LS125
- IC157B1: value ~ -> 74LS08
- IC180B1: value ~ -> 74LS00
- U1, U2: value ~ -> HY5117404B
Changed lines of the file:
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@@
 		(tags "SOIC SO")
 		(property "Reference" "IC180B1"
-			(at 0 0 180)
+			(at 0 0 0)
 			(layer "F.SilkS")
 			(effects
@@
 			)
 		)
-		(property "Value" "~"
+		(property "Value" "74LS00"
 			(at 0 5.28 90)
 			(layer "F.Fab")
@@
 			)
 		)
-		(property "Value" "~"
+		(property "Value" "HY5117404B"
 			(at 0 10.16 90)
 			(layer "F.Fab")
@@
 		(tags "SOIC SO")
 		(property "Reference" "IC157B1"
-			(at 0 0.14 180)
+			(at 0 0.14 0)
 			(layer "F.SilkS")
 			(effects
@@
 			)
 		)
-		(property "Value" "~"
+		(property "Value" "74LS08"
 			(at 0 5.28 90)
 			(layer "F.Fab")
-			(hide yes)
 			(effects
 				(font
@@
 			)
 		)
-		(property "Value" "~"
+		(property "Value" "74LS125"
 			(at 0 5.28 90)
 			(layer "F.Fab")
@@
 			)
 		)
-		(property "Value" "~"
+		(property "Value" "HY5117404B"
 			(at 0 10.16 90)
 			(layer "F.Fab")
@@
 			)
 		)
-		(property "Value" "~"
+		(property "Value" "74LS125"
 			(at 0 5.28 90)
 			(layer "F.Fab")
@@
 			(at 0 5.9 90)
 			(layer "F.Fab")
-			(hide yes)
 			(effects
 				(font
@@
 			)
 		)
-		(property "Value" "~"
+		(property "Value" "74LS125"
 			(at 0 5.28 90)
 			(layer "F.Fab")
