File: KICAD/4mb mapper nms8280.kicad_sch (KiCad schematic)
At the start: 22 parts, among them IC147 74LS157, IC147B1 74LS157, IC149 74LS670, IC149B1 74LS670, J1 Conn_01x10_Pin

Commit message: Update IC147 footprints to SOIC-16
Parts:
- IC147, IC147B1: footprint Package_SO:SOIC-16W_5.3x10.2mm_P1.27mm -> Package_SO:SOIC-16_3.9x9.9mm_P1.27mm
Changed lines of the file:
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@@
 			)
 		)
-		(property "Footprint" "Package_SO:SOIC-16W_5.3x10.2mm_P1.27mm"
+		(property "Footprint" "Package_SO:SOIC-16_3.9x9.9mm_P1.27mm"
 			(at 242.57 36.83 0)
 			(hide yes)
@@
 			)
 		)
-		(property "Footprint" "Package_SO:SOIC-16W_5.3x10.2mm_P1.27mm"
+		(property "Footprint" "Package_SO:SOIC-16_3.9x9.9mm_P1.27mm"
 			(at 208.28 36.83 0)
 			(hide yes)
