File: KICAD/4mb mapper nms8280.kicad_pcb (KiCad board)
At the start: 2 copper layers, 102.2 x 68.2 mm, 28 parts, among them IC131 74LS125, IC131B1 74LS125, IC131C1 74LS125, IC147 74LS157, IC147B1 74LS157, IC149 74LS670, IC149B1 74LS670, IC157B1 74LS08, IC180B1 74LS00, J1 Conn_01x10_Pin, U1 HY5117404B, U2 HY5117404B

Commit message: Update IC147 footprints to SOIC-16
Parts:
- IC131, IC131B1, IC131C1: value 74LS125 -> ~
- IC147, IC147B1: footprint Package_SO:SOIC-16W_5.3x10.2mm_P1.27mm -> Package_SO:SOIC-16_3.9x9.9mm_P1.27mm
- IC157B1: value 74LS08 -> ~
- IC180B1: value 74LS00 -> ~
- U1, U2: value HY5117404B -> ~
- moved C147B1 0.83 mm to (133.8, 98.3)
- moved C147 0.78 mm to (134.1, 86.5)
- renumbered C131C1 to C131B2
Routing:
- net Net-(IC147B1-I0d): track 2.54 -> 4.15 mm
- net A10_IC147B_P7: track 35.6 -> 34.9 mm
- net Net-(IC131B1-4D): track 77.2 -> 77.7 mm

Commit message: Update component values and BOM
Parts:
- CONN131: value ~ -> Pin Header 2x7 2,54mm Rounded
- CONN133, CONN134: value ~ -> Pin Header 2x9 2,54mm Rounded
- CONN147, CONN149: value ~ -> Pin Header 2x8 2,54mm Rounded
- IC131, IC131B1, IC131C1: value ~ -> 74LS125
- IC157B1: value ~ -> 74LS08
- IC180B1: value ~ -> 74LS00
- U1, U2: value ~ -> HY5117404B
Changed lines of the file:
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@@
 			)
 		)
-		(property "Value" "~"
+		(property "Value" "74LS00"
 			(at 0 5.28 90)
 			(layer "F.Fab")
@@
 			)
 		)
-		(property "Value" "~"
+		(property "Value" "HY5117404B"
 			(at 0 10.16 90)
 			(layer "F.Fab")
@@
 			)
 		)
-		(property "Value" "~"
+		(property "Value" "74LS08"
 			(at 0 5.28 90)
 			(layer "F.Fab")
@@
 			)
 		)
-		(property "Value" "~"
+		(property "Value" "74LS125"
 			(at 0 5.28 90)
 			(layer "F.Fab")
@@
 			)
 		)
-		(property "Value" "~"
+		(property "Value" "HY5117404B"
 			(at 0 10.16 90)
 			(layer "F.Fab")
@@
 			)
 		)
-		(property "Value" "~"
+		(property "Value" "74LS125"
 			(at 0 5.28 90)
 			(layer "F.Fab")
@@
 			)
 		)
-		(property "Value" "~"
+		(property "Value" "74LS125"
 			(at 0 5.28 90)
 			(layer "F.Fab")
@@
 			)
 		)
-		(property "Value" "~"
+		(property "Value" "Pin Header 2x9 2,54mm Rounded"
 			(at 1.27 -22.7 90)
 			(layer "B.Fab")
@@
 			)
 		)
-		(property "Value" "~"
+		(property "Value" "Pin Header 2x9 2,54mm Rounded"
 			(at 1.27 -22.7 90)
 			(layer "B.Fab")
@@
 			)
 		)
-		(property "Value" "~"
+		(property "Value" "Pin Header 2x7 2,54mm Rounded"
 			(at 1.27 -17.62 90)
 			(layer "B.Fab")
@@
 			)
 		)
-		(property "Value" "~"
+		(property "Value" "Pin Header 2x8 2,54mm Rounded"
 			(at 1.27 -20.16 90)
 			(layer "B.Fab")
@@
 			)
 		)
-		(property "Value" "~"
+		(property "Value" "Pin Header 2x8 2,54mm Rounded"
 			(at 1.27 -20.16 90)
 			(layer "B.Fab")
